File: FlashCartProgrammer/KiCad/FlashCartProgrammer.kicad_sch (KiCad schematic)
At the start: 85 parts, among them J1 Vic20 Cartridge Connector, J10 Vic20 Header, J11 ZIF Header, J2 C64 Cartridge Connector, J3 +5V, J4 USB_A_KeyBoard, J5 BOOT SEL, J6 VGA, J7 DM3D-SF, J8 SWD, J9 C64 Header, U1 TLV74311PDBVR, U10 27C400, U2 TLV74333PDBVR, U3 W25Q16JVSSIQ, U4 RP2350B-QFN80, U5 74LS573, U6 74LS573, U7 TXS0108EPW, U8 TXS0108EPW, U9 TXS0108EPW, Y1 12MHz

Commit message: - Updated to KiCad 10.
Parts:
- J4: footprint Connector_USB:USB_A_Molex_67643_Horizontal -> Connector_USB:USB_A_Connfly_DS1095
- U10: footprint Socket:DIP_Socket-40_W11.9_W12.7_W15.24_W17.78_W18.5_3M_240-1280-00-0602J -> Socket:DIP_Socket-40_W11.9mm_W12.7mm_W15.24mm_W17.78mm_W18.5mm_3M_240-1280-00-0602J
Connections:
- net GND: now also J4.SH (Shield), J6.SH; no longer J4.5 (Shield), J6.0
- net SPI1.~{CS} renamed SPI1.CS
