File: FlashCartProgrammer/KiCad/FlashCartProgrammer.kicad_sch (KiCad schematic)
At the start: 85 parts, among them J1 Vic20_Cartridge_Connector, J10 Vic20 Header, J11 ZIF Header, J2 c64-Cartridge-Connector, J3 +5V, J4 USB_A_KeyBoard, J5 BOOT SEL, J6 DE15_Socket_HighDensity_Mount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, J7 DM3D-SF, J8 SWD, J9 C64 Header, U1 TLV74311PDBVR, U10 27C400, U18 74LS245, U2 TLV74333PDBVR, U3 W25Q16JVSSIQ, U4 RP2354B-QFN80, U5 74LS573, U6 74LS573, U7 TXS0108EPW, U8 TXS0108EPW, Y1 12MHz

Commit message: - Added support for larger flash roms. - Increased the hole size for the ZIF socket. - Regenerated the ibom and gerber files.
Parts:
- removed H1, H2: MountingHole_Pad, MountingHole:MountingHole_3.5mm, symbol Mechanical:MountingHole
- C19, R11, U3: Note (none) -> DNP
- J10: value Vic20 Header -> Vic20
- J11: value ZIF Header -> ZIF
- J9: value C64 Header -> C64
Connections:
- net A19: now also J10.8 (Pin_8), J9.6 (Pin_6)
- no-connect marks 48 -> 46
Changed lines of the file:
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@@
 		(comment 1 "Fixed the patch wires required on Rev B")
 		(comment 2 "Added reset pin to ZIF Header.")
+		(comment 3 "Added A19 to both C64 and VIC Headers.")
 	)
 	(text "VGA_ID_BIT1"
@@
 	)
 	(no_connect
-		(at 383.54 243.84)
-	)
-	(no_connect
 		(at 454.66 297.18)
 	)
 	(no_connect
-		(at 383.54 274.32)
-	)
-	(no_connect
 		(at 454.66 287.02)
 	)
@@
 	)
 	(bus_entry
+		(at 398.78 243.84)
+		(size 2.54 -2.54)
+		(stroke
+			(width 0)
+			(type default)
+		)
+	)
+	(bus_entry
 		(at 218.44 139.7)
 		(size -2.54 -2.54)
@@
 	)
 	(bus_entry
+		(at 398.78 274.32)
+		(size 2.54 2.54)
+		(stroke
+			(width 0)
+			(type default)
+		)
+	)
+	(bus_entry
 		(at 398.78 284.48)
 		(size 2.54 2.54)
@@
 	(wire
 		(pts
+			(xy 398.78 243.84) (xy 383.54 243.84)
+		)
+		(stroke
+			(width 0)
+			(type default)
+		)
+	)
+	(wire
+		(pts
 			(xy 50.8 78.74) (xy 50.8 81.28)
 		)
@@
 	(wire
 		(pts
-			(xy 383.54 269.24) (xy 388.62 269.24)
+			(xy 383.54 269.24) (xy 386.08 269.24)
 		)
 		(stroke
@@
 	(wire
 		(pts
-			(xy 383.54 271.78) (xy 388.62 271.78)
+			(xy 383.54 271.78) (xy 386.08 271.78)
 		)
 		(stroke
@@
 	(bus
 		(pts
+			(xy 401.32 238.76) (xy 401.32 279.4)
+		)
+		(stroke
+			(width 0)
+			(type default)
+		)
+	)
+	(bus
+		(pts
 			(xy 218.44 139.7) (xy 218.44 142.24)
 		)
@@
 	(wire
 		(pts
-			(xy 383.54 248.92) (xy 388.62 248.92)
+			(xy 383.54 248.92) (xy 386.08 248.92)
 		)
 		(stroke
@@
 		)
 	)
-	(bus
+	(wire
 		(pts
-			(xy 401.32 238.76) (xy 401.32 279.4)
+			(xy 495.3 274.32) (xy 495.3 276.86)
 		)
 		(stroke
@@
 	(wire
 		(pts
-			(xy 495.3 274.32) (xy 495.3 276.86)
+			(xy 541.02 251.46) (xy 520.7 251.46)
 		)
 		(stroke
@@
 	(wire
 		(pts
-			(xy 541.02 251.46) (xy 520.7 251.46)
+			(xy 500.38 241.3) (xy 477.52 241.3)
 		)
 		(stroke
@@
 	(wire
 		(pts
-			(xy 500.38 241.3) (xy 477.52 241.3)
+			(xy 403.86 203.2) (xy 424.18 203.2)
 		)
 		(stroke
@@
 	(wire
 		(pts
-			(xy 403.86 203.2) (xy 424.18 203.2)
+			(xy 454.66 274.32) (xy 462.28 274.32)
 		)
 		(stroke
@@
 	(wire
 		(pts
-			(xy 454.66 274.32) (xy 462.28 274.32)
+			(xy 383.54 274.32) (xy 398.78 274.32)
 		)
 		(stroke
@@
 	(wire
 		(pts
-			(xy 383.54 246.38) (xy 388.62 246.38)
+			(xy 383.54 246.38) (xy 386.08 246.38)
 		)
 		(stroke
@@
 		)
 	)
+	(label "A19"
+		(at 396.24 243.84 180)
+		(effects
+			(font
+				(size 1.27 1.27)
+			)
+			(justify right bottom)
+		)
+	)
 	(label "D13"
 		(at 490.22 302.26 0)
@@
 		)
 	)
+	(label "A19"
+		(at 396.24 274.32 180)
+		(effects
+			(font
+				(size 1.27 1.27)
+			)
+			(justify right bottom)
+		)
+	)
 	(label "2350_USB_D-"
 		(at 218.44 81.28 180)
@@
 	(global_label "~{OE}"
 		(shape input)
-		(at 388.62 248.92 0)
+		(at 386.08 248.92 0)
 		(fields_autoplaced yes)
 		(effects
@@
 		)
 		(property "Intersheetrefs" "${INTERSHEET_REFS}"
-			(at 394.0847 248.92 0)
+			(at 391.5447 248.92 0)
 			(hide yes)
 			(show_name no)
@@
 	(global_label "~{WE}"
 		(shape input)
-		(at 388.62 271.78 0)
+		(at 386.08 271.78 0)
 		(fields_autoplaced yes)
 		(effects
@@
 		)
 		(property "Intersheetrefs" "${INTERSHEET_REFS}"
-			(at 394.2056 271.78 0)
+			(at 391.6656 271.78 0)
 			(hide yes)
 			(show_name no)
@@
 	(global_label "~{WE}"
 		(shape input)
-		(at 388.62 246.38 0)
+		(at 386.08 246.38 0)
 		(fields_autoplaced yes)
 		(effects
@@
 		)
 		(property "Intersheetrefs" "${INTERSHEET_REFS}"
-			(at 394.2056 246.38 0)
+			(at 391.6656 246.38 0)
 			(hide yes)
 			(show_name no)
@@
 	(global_label "~{OE}"
 		(shape input)
-		(at 388.62 269.24 0)
+		(at 386.08 269.24 0)
 		(fields_autoplaced yes)
 		(effects
@@
 		)
 		(property "Intersheetrefs" "${INTERSHEET_REFS}"
-			(at 394.0847 269.24 0)
+			(at 391.5447 269.24 0)
 			(hide yes)
 			(show_name no)
@@
 			)
 		)
-		(property "Value" "ZIF Header"
+		(property "Value" "ZIF"
 			(at 376.949 164.9593 90)
 			(hide yes)
@@
 			)
 		)
-		(property "Value" "Vic20 Header"
+		(property "Value" "Vic20"
 			(at 376.949 236.0793 90)
 			(show_name no)
@@
 	)
 	(symbol
-		(lib_id "Mechanical:MountingHole")
-		(at 444.5 398.78 0)
-		(unit 1)
-		(body_style 1)
-		(exclude_from_sim no)
-		(in_bom no)
-		(on_board yes)
-		(in_pos_files yes)
-		(dnp no)
-		(property "Reference" "H2"
-			(at 447.04 397.5099 0)
-			(show_name no)
-			(do_not_autoplace no)
-			(effects
-				(font
-					(size 1.27 1.27)
-				)
-				(justify left)
-			)
-		)
-		(property "Value" "MountingHole_Pad"
-			(at 447.04 400.0499 0)
-			(show_name no)
-			(do_not_autoplace no)
-			(effects
-				(font
-					(size 1.27 1.27)
-				)
-				(justify left)
-			)
-		)
-		(property "Footprint" "MountingHole:MountingHole_3.5mm"
-			(at 444.5 398.78 0)
-			(hide yes)
-			(show_name no)
-			(do_not_autoplace no)
-			(effects
-				(font
-					(size 1.27 1.27)
-				)
-			)
-		)
-		(property "Datasheet" ""
-			(at 444.5 398.78 0)
-			(hide yes)
-			(show_name no)
-			(do_not_autoplace no)
-			(effects
-				(font
-					(size 1.27 1.27)
-				)
-			)
-		)
-		(property "Description" "Mounting Hole without connection"
-			(at 444.5 398.78 0)
-			(hide yes)
-			(show_name no)
-			(do_not_autoplace no)
-			(effects
-				(font
-					(size 1.27 1.27)
-				)
-			)
-		)
-		(instances
-			(project "FlashCartProgrammer"
-				(path "/26813dea-ac31-4359-98cd-29d1f4f9df4c"
-					(reference "H2")
-					(unit 1)
-				)
-			)
-		)
-	)
-	(symbol
 		(lib_id "power:PWR_FLAG")
 		(at 441.96 30.48 0)
@@
 			)
 		)
-		(property "Value" "C64 Header"
+		(property "Value" "C64"
 			(at 375.92 279.4 90)
 			(show_name no)
@@
 			)
 		)
-		(property "Note" ""
+		(property "Note" "DNP"
 			(at 27.94 88.9 0)
-			(hide yes)
 			(show_name no)
 			(do_not_autoplace no)
@@
 			)
 		)
-		(property "Note" ""
+		(property "Note" "DNP"
 			(at 35.56 109.22 0)
-			(hide yes)
 			(show_name no)
 			(do_not_autoplace no)
@@
 			)
 		)
-		(property "Note" ""
+		(property "Note" "DNP"
 			(at 50.8 83.82 0)
-			(hide yes)
 			(show_name no)
 			(do_not_autoplace no)
@@
 					(unit 1)
 				)
-			)
-		)
-	)
-	(symbol
-		(lib_id "Mechanical:MountingHole")
-		(at 444.5 393.7 0)
-		(unit 1)
-		(body_style 1)
-		(exclude_from_sim no)
-		(in_bom no)
-		(on_board yes)
-		(in_pos_files yes)
-		(dnp no)
-		(property "Reference" "H1"
-			(at 447.04 392.4299 0)
-			(show_name no)
-			(do_not_autoplace no)
-			(effects
-				(font
-					(size 1.27 1.27)
-				)
-				(justify left)
-			)
-		)
-		(property "Value" "MountingHole_Pad"
-			(at 447.04 394.9699 0)
-			(show_name no)
-			(do_not_autoplace no)
-			(effects
-				(font
-					(size 1.27 1.27)
-				)
-				(justify left)
-			)
-		)
-		(property "Footprint" "MountingHole:MountingHole_3.5mm"
-			(at 444.5 393.7 0)
-			(hide yes)
-			(show_name no)
-			(do_not_autoplace no)
-			(effects
-				(font
-					(size 1.27 1.27)
-				)
-			)
-		)
-		(property "Datasheet" ""
-			(at 444.5 393.7 0)
-			(hide yes)
-			(show_name no)
-			(do_not_autoplace no)
-			(effects
-				(font
-					(size 1.27 1.27)
-				)
-			)
-		)
-		(property "Description" "Mounting Hole without connection"
-			(at 444.5 393.7 0)
-			(hide yes)
-			(show_name no)
-			(do_not_autoplace no)
-			(effects
-				(font
-					(size 1.27 1.27)
-				)
-			)
-		)
-		(instances
-			(project "FlashCartProgrammer"
-				(path "/26813dea-ac31-4359-98cd-29d1f4f9df4c"
-					(reference "H1")
-					(unit 1)
-				)
