File: FlashCartProgrammer/KiCad/FlashCartProgrammer.kicad_pcb (KiCad board)
At the start: 2 copper layers, 100 x 100 mm, 85 parts, among them J1 Vic20_Cartridge_Connector, J10 Vic20 Header, J11 ZIF Header, J2 c64-Cartridge-Connector, J3 +5V, J4 USB_A_KeyBoard, J5 BOOT SEL, J6 DE15_Socket_HighDensity_Mount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, J7 DM3D-SF, J8 SWD, J9 C64 Header, U1 TLV74311PDBVR, U10 27C400, U18 74LS245, U2 TLV74333PDBVR, U3 W25Q16JVSSIQ, U4 RP2354B-QFN80, U5 74LS573, U6 74LS573, U7 TXS0108EPW, U8 TXS0108EPW, Y1 12MHz

Commit message: - Added support for larger flash roms. - Increased the hole size for the ZIF socket. - Regenerated the ibom and gerber files.
Parts:
- removed H1, H2: MountingHole_Pad, MountingHole:MountingHole_3.5mm
- J10: value Vic20 Header -> Vic20
- J11: value ZIF Header -> ZIF
- J9: value C64 Header -> C64
- R11, R13, R26: moved to B.Cu
- moved R26 11.2 mm to (125.9, 115.4), turned to -90 degrees
- moved J6 4.02 mm to (187.1, 81.5)
- moved R10 4.02 mm to (183.5, 81.5)
- moved R12 4.02 mm to (183.5, 83.8)
- moved R14 4.02 mm to (183.5, 86.0)
- moved J4 2.40 mm to (183.8, 137.0)
- moved C6 1.24 mm to (178.0, 138.3)
Connections:
- J10 pad 8: unconnected-(J10-Pin_8-Pad8) -> /A19
- J9 pad 6: unconnected-(J9-Pin_6-Pad6) -> /A19
Routing:
- net /A19: track 89.5 -> 139.1 mm
- net /D0: track 164.0 -> 185.7 mm
- net /D1: track 163.5 -> 182.5 mm, vias 2 -> 3
- net /D4: track 160.7 -> 176.1 mm
- net /D5: track 156.3 -> 169.4 mm
- net GND: track 98.5 -> 110.1 mm, vias 130 -> 172
- net /2350_QSPI.~{CS}: track 41.1 -> 51.8 mm, vias 2 -> 3
- net /A5: track 92.4 -> 102.5 mm, vias 2 -> 3
- net /D3: track 175.7 -> 184.3 mm
- net /A16: track 107.2 -> 115.5 mm, vias 3 -> 1
- net /D6: track 152.4 -> 160.5 mm
- net /A17: track 118.1 -> 124.6 mm, vias 2 -> 0
- net ~{WE}: track 121.4 -> 115.4 mm, vias 0 -> 1
- net 3v3_DATA_OE: track 55.9 -> 50.2 mm
- net /D2: track 177.8 -> 183.3 mm
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Other:
- board text added: "A13"
- board text added: "A14"
- board text added: "A15"
- board text added: "A16"
- board text added: "A17"
- board text added: "A18"
- board text added: "A19"
- board text added: "N.C"
- board text added: "~{OE}"
- board text added: "~{RST}"
- board text added: "~{WE}"
